File: Atari Joystick Tester.sch (KiCad schematic (older format))
At the start: 24 parts, among them J1 Atari_Joystick, J2 Paddle A, J3 Paddle B, J4 Barrel_Jack, J5 Mount, J6 Mount, J7 Mount, J8 Mount, SW1 PADDLE A SEL., SW2 PADDLE B SEL.

Commit message: Reoriented components.
Parts:
- D1, D2, D3, D4, D5, D6, D7: footprint (none) -> LEDs:LED_D5.0mm
- J1: footprint (none) -> RND_DSUB:DSUB-9_Male_Vertical_Pitch2.77x2.84mm
- J2, J3: footprint (none) -> Connectors_Terminal_Blocks:TerminalBlock_bornier-2_P5.08mm
- J4: footprint (none) -> Connectors:BARREL_JACK
- J5, J6, J7, J8: footprint (none) -> mounting:1pin
- R1, R2, R3, R4, R5, R6, R7: footprint (none) -> Resistors_THT:R_Axial_DIN0207_L6.3mm_D2.5mm_P10.16mm_Horizontal
- SW1, SW2: footprint (none) -> Pin_Headers:Pin_Header_Straight_1x03_Pitch2.54mm
Changed lines of the file:
@@
 F 0 "D1" H 2750 3800 50  0000 C CNN
 F 1 "UP" H 2750 3600 50  0000 C CNN
-F 2 "" H 2750 3700 50  0001 C CNN
+F 2 "LEDs:LED_D5.0mm" H 2750 3700 50  0001 C CNN
 F 3 "" H 2750 3700 50  0001 C CNN
 	1    2750 3700
@@
 F 0 "D2" H 3050 3800 50  0000 C CNN
 F 1 "DOWN" H 3050 3600 50  0000 C CNN
-F 2 "" H 3050 3700 50  0001 C CNN
+F 2 "LEDs:LED_D5.0mm" H 3050 3700 50  0001 C CNN
 F 3 "" H 3050 3700 50  0001 C CNN
 	1    3050 3700
@@
 F 0 "D3" H 3350 3800 50  0000 C CNN
 F 1 "LEFT" H 3350 3600 50  0000 C CNN
-F 2 "" H 3350 3700 50  0001 C CNN
+F 2 "LEDs:LED_D5.0mm" H 3350 3700 50  0001 C CNN
 F 3 "" H 3350 3700 50  0001 C CNN
 	1    3350 3700
@@
 F 0 "D4" H 3650 3800 50  0000 C CNN
 F 1 "RIGHT" H 3650 3600 50  0000 C CNN
-F 2 "" H 3650 3700 50  0001 C CNN
+F 2 "LEDs:LED_D5.0mm" H 3650 3700 50  0001 C CNN
 F 3 "" H 3650 3700 50  0001 C CNN
 	1    3650 3700
@@
 F 0 "D5" H 3950 3800 50  0000 C CNN
 F 1 "FIRE 0" H 3950 3600 50  0000 C CNN
-F 2 "" H 3950 3700 50  0001 C CNN
+F 2 "LEDs:LED_D5.0mm" H 3950 3700 50  0001 C CNN
 F 3 "" H 3950 3700 50  0001 C CNN
 	1    3950 3700
@@
 F 0 "D6" H 4600 3800 50  0000 C CNN
 F 1 "FIRE 1" H 4600 3600 50  0000 C CNN
-F 2 "" H 4600 3700 50  0001 C CNN
+F 2 "LEDs:LED_D5.0mm" H 4600 3700 50  0001 C CNN
 F 3 "" H 4600 3700 50  0001 C CNN
 	1    4600 3700
@@
 F 0 "D7" H 5300 3800 50  0000 C CNN
 F 1 "FIRE 2" H 5300 3600 50  0000 C CNN
-F 2 "" H 5300 3700 50  0001 C CNN
+F 2 "LEDs:LED_D5.0mm" H 5300 3700 50  0001 C CNN
 F 3 "" H 5300 3700 50  0001 C CNN
 	1    5300 3700
@@
 F 0 "J1" H 3650 7000 50  0000 C CNN
 F 1 "Atari_Joystick" H 3650 5875 50  0000 C CNN
-F 2 "" H 3650 6450 50  0001 C CNN
+F 2 "RND_DSUB:DSUB-9_Male_Vertical_Pitch2.77x2.84mm" H 3650 6450 50  0001 C CNN
 F 3 "" H 3650 6450 50  0001 C CNN
 	1    3650 6450
@@
 F 0 "R1" V 2830 4100 50  0000 C CNN
 F 1 "330" V 2750 4100 50  0000 C CNN
-F 2 "" V 2680 4100 50  0001 C CNN
+F 2 "Resistors_THT:R_Axial_DIN0207_L6.3mm_D2.5mm_P10.16mm_Horizontal" V 2680 4100 50  0001 C CNN
 F 3 "" H 2750 4100 50  0001 C CNN
 	1    2750 4100
@@
 F 0 "R2" V 3130 4100 50  0000 C CNN
 F 1 "330" V 3050 4100 50  0000 C CNN
-F 2 "" V 2980 4100 50  0001 C CNN
+F 2 "Resistors_THT:R_Axial_DIN0207_L6.3mm_D2.5mm_P10.16mm_Horizontal" V 2980 4100 50  0001 C CNN
 F 3 "" H 3050 4100 50  0001 C CNN
 	1    3050 4100
@@
 F 0 "R3" V 3430 4100 50  0000 C CNN
 F 1 "330" V 3350 4100 50  0000 C CNN
-F 2 "" V 3280 4100 50  0001 C CNN
+F 2 "Resistors_THT:R_Axial_DIN0207_L6.3mm_D2.5mm_P10.16mm_Horizontal" V 3280 4100 50  0001 C CNN
 F 3 "" H 3350 4100 50  0001 C CNN
 	1    3350 4100
@@
 F 0 "R4" V 3730 4100 50  0000 C CNN
 F 1 "330" V 3650 4100 50  0000 C CNN
-F 2 "" V 3580 4100 50  0001 C CNN
+F 2 "Resistors_THT:R_Axial_DIN0207_L6.3mm_D2.5mm_P10.16mm_Horizontal" V 3580 4100 50  0001 C CNN
 F 3 "" H 3650 4100 50  0001 C CNN
 	1    3650 4100
@@
 F 0 "R5" V 4030 4100 50  0000 C CNN
 F 1 "330" V 3950 4100 50  0000 C CNN
-F 2 "" V 3880 4100 50  0001 C CNN
+F 2 "Resistors_THT:R_Axial_DIN0207_L6.3mm_D2.5mm_P10.16mm_Horizontal" V 3880 4100 50  0001 C CNN
 F 3 "" H 3950 4100 50  0001 C CNN
 	1    3950 4100
@@
 F 0 "R6" V 4680 4100 50  0000 C CNN
 F 1 "330" V 4600 4100 50  0000 C CNN
-F 2 "" V 4530 4100 50  0001 C CNN
+F 2 "Resistors_THT:R_Axial_DIN0207_L6.3mm_D2.5mm_P10.16mm_Horizontal" V 4530 4100 50  0001 C CNN
 F 3 "" H 4600 4100 50  0001 C CNN
 	1    4600 4100
@@
 F 0 "R7" V 5380 4100 50  0000 C CNN
 F 1 "330" V 5300 4100 50  0000 C CNN
-F 2 "" V 5230 4100 50  0001 C CNN
+F 2 "Resistors_THT:R_Axial_DIN0207_L6.3mm_D2.5mm_P10.16mm_Horizontal" V 5230 4100 50  0001 C CNN
 F 3 "" H 5300 4100 50  0001 C CNN
 	1    5300 4100
@@
 F 0 "J2" H 4700 2350 50  0000 C CNN
 F 1 "Paddle A" H 4700 2050 50  0000 C CNN
-F 2 "" H 4700 2250 50  0001 C CNN
+F 2 "Connectors_Terminal_Blocks:TerminalBlock_bornier-2_P5.08mm" H 4700 2250 50  0001 C CNN
 F 3 "" H 4700 2250 50  0001 C CNN
 	1    4700 2250
@@
 F 0 "J3" H 5400 2350 50  0000 C CNN
 F 1 "Paddle B" H 5400 2050 50  0000 C CNN
-F 2 "" H 5400 2250 50  0001 C CNN
+F 2 "Connectors_Terminal_Blocks:TerminalBlock_bornier-2_P5.08mm" H 5400 2250 50  0001 C CNN
 F 3 "" H 5400 2250 50  0001 C CNN
 	1    5400 2250
@@
 F 0 "SW1" H 4700 5070 50  0000 C CNN
 F 1 "PADDLE A SEL." H 4700 4700 50  0000 C CNN
-F 2 "" H 4700 4900 50  0001 C CNN
+F 2 "Pin_Headers:Pin_Header_Straight_1x03_Pitch2.54mm" H 4700 4900 50  0001 C CNN
 F 3 "" H 4700 4900 50  0001 C CNN
 	1    4700 4900
@@
 F 0 "SW2" H 5400 5070 50  0000 C CNN
 F 1 "PADDLE B SEL." H 5400 4700 50  0000 C CNN
-F 2 "" H 5400 4900 50  0001 C CNN
+F 2 "Pin_Headers:Pin_Header_Straight_1x03_Pitch2.54mm" H 5400 4900 50  0001 C CNN
 F 3 "" H 5400 4900 50  0001 C CNN
 	1    5400 4900
@@
 F 0 "J4" H 1400 1610 50  0000 C CNN
 F 1 "Barrel_Jack" H 1400 1225 50  0000 C CNN
-F 2 "" H 1450 1360 50  0001 C CNN
+F 2 "Connectors:BARREL_JACK" H 1450 1360 50  0001 C CNN
 F 3 "" H 1450 1360 50  0001 C CNN
 	1    1400 1400
@@
 F 0 "J5" H 10500 700 50  0000 C CNN
 F 1 "Mount" H 10300 700 50  0000 C CNN
-F 2 "" H 10400 800 50  0001 C CNN
+F 2 "mounting:1pin" H 10400 800 50  0001 C CNN
 F 3 "" H 10400 800 50  0001 C CNN
 	1    10400 800
@@
 F 0 "J6" H 10700 700 50  0000 C CNN
 F 1 "Mount" H 10500 700 50  0000 C CNN
-F 2 "" H 10600 800 50  0001 C CNN
+F 2 "mounting:1pin" H 10600 800 50  0001 C CNN
 F 3 "" H 10600 800 50  0001 C CNN
 	1    10600 800
@@
 F 0 "J7" H 10900 700 50  0000 C CNN
 F 1 "Mount" H 10700 700 50  0000 C CNN
-F 2 "" H 10800 800 50  0001 C CNN
+F 2 "mounting:1pin" H 10800 800 50  0001 C CNN
 F 3 "" H 10800 800 50  0001 C CNN
 	1    10800 800
@@
 F 0 "J8" H 11100 700 50  0000 C CNN
 F 1 "Mount" H 10900 700 50  0000 C CNN
-F 2 "" H 11000 800 50  0001 C CNN
+F 2 "mounting:1pin" H 11000 800 50  0001 C CNN
 F 3 "" H 11000 800 50  0001 C CNN
 	1    11000 800
